Commit message: atlas and valkyrie are added

File: Simulator/SimulationModel/Valkyrie/valkyrie_sim.urdf (robot description, URDF)
Before this commit: robot valkyrie, 80 links, 79 joints
Links:
- link hokuyo_link: geometry collision box size=0.08 0.06 0.04238; collision cylinder length=0.047 radius=0.024425
- link leftAnklePitchLink: geometry collision mesh filename=meshes/legs/lj5.dae; visual mesh filename=meshes/legs/lj5.dae
- link leftElbowPitchLink: geometry collision mesh filename=meshes/arms/aj4_left.dae; visual mesh filename=meshes/arms/aj4_left.dae
- link leftFoot: geometry collision box size=0.27 0.16 0.064; visual mesh filename=meshes/legs/foot.dae
- link leftForearmLink: geometry collision mesh filename=meshes/arms/aj5_left.dae; visual mesh filename=meshes/arms/aj5_left.dae
- link leftHipPitchLink: geometry collision mesh filename=meshes/legs/lj3_left.dae; visual mesh filename=meshes/legs/lj3_left.dae
- link leftHipRollLink: geometry collision mesh filename=meshes/legs/lj2_left.dae; visual mesh filename=meshes/legs/lj2_left.dae
- link leftHipYawLink: geometry collision mesh filename=meshes/legs/lj1_left.dae; visual mesh filename=meshes/legs/lj1_left.dae
- link leftIndexFingerPitch1Link: geometry collision mesh filename=meshes/fingers/indexj1_left.dae; visual mesh filename=meshes/fingers/indexj1_left.dae
- link leftIndexFingerPitch2Link: geometry collision mesh filename=meshes/fingers/indexj2_left.dae; visual mesh filename=meshes/fingers/indexj2_left.dae
- link leftIndexFingerPitch3Link: geometry collision mesh filename=meshes/fingers/indexj3_left.dae; visual mesh filename=meshes/fingers/indexj3_left.dae
- link leftKneePitchLink: geometry collision mesh filename=meshes/legs/lj4_left.dae; visual mesh filename=meshes/legs/lj4_left.dae
- link leftMiddleFingerPitch1Link: geometry collision mesh filename=meshes/fingers/middlej1_left.dae; visual mesh filename=meshes/fingers/middlej1_left.dae
- link leftMiddleFingerPitch2Link: geometry collision mesh filename=meshes/fingers/middlej2_left.dae; visual mesh filename=meshes/fingers/middlej2_left.dae
- link leftMiddleFingerPitch3Link: geometry collision mesh filename=meshes/fingers/middlej3_left.dae; visual mesh filename=meshes/fingers/middlej3_left.dae
- link leftPalm: geometry collision mesh filename=meshes/arms/palm_left.dae; visual mesh filename=meshes/arms/palm_left.dae
- link leftPinkyPitch1Link: geometry collision mesh filename=meshes/fingers/pinkyj1_left.dae; visual mesh filename=meshes/fingers/pinkyj1_left.dae
- link leftPinkyPitch2Link: geometry collision mesh filename=meshes/fingers/pinkyj2_left.dae; visual mesh filename=meshes/fingers/pinkyj2_left.dae
- link leftPinkyPitch3Link: geometry collision mesh filename=meshes/fingers/pinkyj3_left.dae; visual mesh filename=meshes/fingers/pinkyj3_left.dae
- link leftShoulderPitchLink: geometry collision mesh filename=meshes/arms/aj1_left.dae; visual mesh filename=meshes/arms/aj1_left.dae
- link leftShoulderRollLink: geometry collision mesh filename=meshes/arms/aj2_left.dae; visual mesh filename=meshes/arms/aj2_left.dae
- link leftShoulderYawLink: geometry collision mesh filename=meshes/arms/aj3_left.dae; visual mesh filename=meshes/arms/aj3_left.dae
- link leftThumbPitch1Link: geometry collision mesh filename=meshes/fingers/thumbj2_left.dae; visual mesh filename=meshes/fingers/thumbj2_left.dae
- link leftThumbPitch2Link: geometry collision mesh filename=meshes/fingers/thumbj3_left.dae; visual mesh filename=meshes/fingers/thumbj3_left.dae
- link leftThumbPitch3Link: geometry collision mesh filename=meshes/fingers/thumbj4_left.dae; visual mesh filename=meshes/fingers/thumbj4_left.dae
- link leftThumbRollLink: geometry collision mesh filename=meshes/fingers/thumbj1_left.dae; visual mesh filename=meshes/fingers/thumbj1_left.dae
- link leftWristRollLink: geometry collision mesh filename=meshes/arms/aj6_left.dae; visual mesh filename=meshes/arms/aj6_left.dae
- link lowerNeckPitchLink: geometry collision mesh filename=meshes/head/neckj1.dae; visual mesh filename=meshes/head/neckj1.dae
- link neckYawLink: geometry collision mesh filename=meshes/head/neckj2.dae; visual mesh filename=meshes/head/neckj2.dae
- link pelvis: geometry collision mesh filename=meshes/pelvis/pelvis.dae; visual mesh filename=meshes/pelvis/pelvis.dae
- link rightAnklePitchLink: geometry collision mesh filename=meshes/legs/lj5.dae; visual mesh filename=meshes/legs/lj5.dae
- link rightElbowPitchLink: geometry collision mesh filename=meshes/arms/aj4_right.dae; visual mesh filename=meshes/arms/aj4_right.dae
- link rightFoot: geometry collision box size=0.27 0.16 0.064; visual mesh filename=meshes/legs/foot.dae
- link rightForearmLink: geometry collision mesh filename=meshes/arms/aj5_right.dae; visual mesh filename=meshes/arms/aj5_right.dae
- link rightHipPitchLink: geometry collision mesh filename=meshes/legs/lj3_right.dae; visual mesh filename=meshes/legs/lj3_right.dae
- link rightHipRollLink: geometry collision mesh filename=meshes/legs/lj2_right.dae; visual mesh filename=meshes/legs/lj2_right.dae
- link rightHipYawLink: geometry collision mesh filename=meshes/legs/lj1_right.dae; visual mesh filename=meshes/legs/lj1_right.dae
- link rightIndexFingerPitch1Link: geometry collision mesh filename=meshes/fingers/indexj1_right.dae; visual mesh filename=meshes/fingers/indexj1_right.dae
- link rightIndexFingerPitch2Link: geometry collision mesh filename=meshes/fingers/indexj2_right.dae; visual mesh filename=meshes/fingers/indexj2_right.dae
- link rightIndexFingerPitch3Link: geometry collision mesh filename=meshes/fingers/indexj3_right.dae; visual mesh filename=meshes/fingers/indexj3_right.dae
- link rightKneePitchLink: geometry collision mesh filename=meshes/legs/lj4_right.dae; visual mesh filename=meshes/legs/lj4_right.dae
- link rightMiddleFingerPitch1Link: geometry collision mesh filename=meshes/fingers/middlej1_right.dae; visual mesh filename=meshes/fingers/middlej1_right.dae
- link rightMiddleFingerPitch2Link: geometry collision mesh filename=meshes/fingers/middlej2_right.dae; visual mesh filename=meshes/fingers/middlej2_right.dae
- link rightMiddleFingerPitch3Link: geometry collision mesh filename=meshes/fingers/middlej3_right.dae; visual mesh filename=meshes/fingers/middlej3_right.dae
- link rightPalm: geometry collision mesh filename=meshes/arms/palm_right.dae; visual mesh filename=meshes/arms/palm_right.dae
- link rightPinkyPitch1Link: geometry collision mesh filename=meshes/fingers/pinkyj1_right.dae; visual mesh filename=meshes/fingers/pinkyj1_right.dae
- link rightPinkyPitch2Link: geometry collision mesh filename=meshes/fingers/pinkyj2_right.dae; visual mesh filename=meshes/fingers/pinkyj2_right.dae
- link rightPinkyPitch3Link: geometry collision mesh filename=meshes/fingers/pinkyj3_right.dae; visual mesh filename=meshes/fingers/pinkyj3_right.dae
- link rightShoulderPitchLink: geometry collision mesh filename=meshes/arms/aj1_right.dae; visual mesh filename=meshes/arms/aj1_right.dae
- link rightShoulderRollLink: geometry collision mesh filename=meshes/arms/aj2_right.dae; visual mesh filename=meshes/arms/aj2_right.dae
- link rightShoulderYawLink: geometry collision mesh filename=meshes/arms/aj3_right.dae; visual mesh filename=meshes/arms/aj3_right.dae
- link rightThumbPitch1Link: geometry collision mesh filename=meshes/fingers/thumbj2_right.dae; visual mesh filename=meshes/fingers/thumbj2_right.dae
- link rightThumbPitch2Link: geometry collision mesh filename=meshes/fingers/thumbj3_right.dae; visual mesh filename=meshes/fingers/thumbj3_right.dae
- link rightThumbPitch3Link: geometry collision mesh filename=meshes/fingers/thumbj4_right.dae; visual mesh filename=meshes/fingers/thumbj4_right.dae
- link rightThumbRollLink: geometry collision mesh filename=meshes/fingers/thumbj1_right.dae; visual mesh filename=meshes/fingers/thumbj1_right.dae
- link rightWristRollLink: geometry collision mesh filename=meshes/arms/aj6_right.dae; visual mesh filename=meshes/arms/aj6_right.dae
- link torso: geometry collision mesh filename=meshes/torso/torso.dae; visual mesh filename=meshes/torso/torso.dae
- link torsoPitchLink: geometry collision mesh filename=meshes/torso/torsopitch.dae; visual mesh filename=meshes/torso/torsopitch.dae
- link torsoYawLink: geometry collision mesh filename=meshes/torso/torsoyaw.dae; visual mesh filename=meshes/torso/torsoyaw.dae
- link upperNeckPitchLink: geometry collision mesh filename=meshes/head/head_multisense_no_visor.dae; visual mesh filename=meshes/head/head_multisense_no_visor.dae
