Commit message: configure correct posture of each linkage of Mercury

File: Simulator/SimulationModel/Mercury_Model/mercury_srlib.urdf (robot description, URDF)
Before this commit: robot mercury, 23 links, 22 joints
Links:
- link thigh_r: geometry visual mesh filename=meshes/color_thigh_R.dae scale=0.001 0.001 0.001

File: Simulator/SimulationModel/Mercury_Model/mercury_srlib_ori.urdf (robot description, URDF)
Before this commit: robot mercury, 21 links, 20 joints
Links:
- added link lleg_led4, mass 0.000000000001
- added link rleg_led4, mass 0.000000000001
- link body: mass 9.5 -> 8.0
Joints:
- added joint fixed_led10: type fixed, parent shank_l, child lleg_led4, origin xyz=0.0 -0.033 -0.47 rpy=0 0 0, axis 0 1 0
- added joint fixed_led5: type fixed, parent shank_r, child rleg_led4, origin xyz=0.0 0.025 -0.47 rpy=0 0 0, axis 0 1 0
- joint abduct_l_to_thigh_l_j: origin xyz=0.0 0.0 -0.03535 rpy=0.0 0 0.01 -> xyz=0.0 0.0 -0.03535 rpy=-0.017 0 0.01
- joint abduct_r_to_thigh_r_j: origin xyz=0.0 0.0 -0.03535 rpy=0.015 0.0 -0.02 -> xyz=0.0 0.0 -0.03535 rpy=0.01 0.0 0.0
- joint ankle_l: origin xyz=0.0 -0.0165 -0.47 rpy=0 0 0 -> xyz=0.0 -0.008 -0.47 rpy=0 0 0
- joint fixed_led2: origin xyz=0.075 0.005 -0.42 rpy=0 0 0 -> xyz=0.075 0.0 -0.42 rpy=0 0 0
- joint fixed_led3: origin xyz=0.0 -0.02 -0.060 rpy=0 0 0 -> xyz=0.035 -0.0 -0.050 rpy=0 0 0
- joint fixed_led4: origin xyz=0.0 -0.0365 -0.47 rpy=0 0 0 -> xyz=0.0 -0.025 -0.47 rpy=0 0 0
- joint fixed_led7: origin xyz=0.075 -0.005 -0.42 rpy=0 0 0 -> xyz=0.075 0.0 -0.42 rpy=0 0 0
- joint fixed_led8: origin xyz=0.0 0.02 -0.062 rpy=0 0 0 -> xyz=0.04 0.0 -0.045 rpy=0 0 0
- joint fixed_led9: origin xyz=0.0 0.02 -0.47 rpy=0 0 0 -> xyz=0.0 0.017 -0.47 rpy=0 0 0
- joint thigh_l_to_knee_l_j: origin xyz=0.0181 -0.005 -0.4575 rpy= 0.008 0 0.00 -> xyz=0.0181 -0.005 -0.4575 rpy= 0.0 0 0.00
- joint thigh_r_to_knee_r_j: origin xyz=0.0181 0.005 -0.4575 rpy=0.02 0 0.04 -> xyz=0.0181 0.005 -0.4575 rpy=0.02 0 0.02

Commit message: Mercury torso.obj updated

File: Simulator/SimulationModel/Mercury_Model/mercury_srlib.urdf (robot description, URDF)
Before this commit: robot mercury, 23 links, 22 joints
Links:
- link body: geometry visual mesh filename=meshes/color_torso.obj scale=0.118 0.118 0.118

Commit message: mercury urdf foot position updated

File: Simulator/SimulationModel/Mercury_Model/mercury_srlib.urdf (robot description, URDF)
Before this commit: robot mercury, 23 links, 22 joints
Links:
- link lfoot: geometry collision box size=0.2 0.01 0.01; visual mesh filename=meshes/color_foot_L.obj scale=1 1 1
- link rfoot: geometry collision box size=0.2 0.01 0.01; visual mesh filename=meshes/color_foot_R.obj scale=1 1 1

Commit message: white torso added in simulation

File: Simulator/SimulationModel/Mercury_Model/mercury_srlib.urdf (robot description, URDF)
Before this commit: robot mercury, 23 links, 22 joints
Links:
- link body: geometry visual mesh filename=meshes/white_torso.obj scale=0.508 0.508 0.508
